File: mspm0-dev-hw/mspm0-dev.kicad_pcb (KiCad board)
At the start: 2 copper layers, 60 x 30 mm, 40 parts, among them J1 USB_C_Receptacle_USB2.0_14P, J2 Conn_02x05_Odd_Even, J3 TC2030, U1 MSPM0G3507SPTR, U4 SPX3819M5-L-3-3, U5 CH340E, Y1 8MHz

Commit message: begin routing
Parts:
- removed C3: 470n, Capacitor_SMD:C_0603_1608Metric
- moved FID2 78.0 mm to (144.0, 104.0)
- moved FID1 69.1 mm to (146.0, 83.0)
- moved FID3 50.7 mm to (100.0, 104.0)
- moved C4 37.6 mm to (109.6, 81.7), turned to -90 degrees
- moved C14 33.8 mm to (121.3, 92.4), turned to -90 degrees
- moved C15 31.6 mm to (119.2, 92.2), turned to -90 degrees
- moved C6 30.3 mm to (116.8, 81.7), turned to -90 degrees
- moved C12 28.3 mm to (129.0, 83.8), turned to 180 degrees
- moved C5 24.7 mm to (113.2, 84.7), turned to 180 degrees
- moved R7 22.1 mm to (129.0, 85.6), turned to 180 degrees
- moved R5 21.6 mm to (134.8, 79.0), turned to -90 degrees
- moved C16 17.9 mm to (133.0, 79.0), turned to 90 degrees
- moved R2 17.3 mm to (98.0, 100.0)
- moved R3 9.13 mm to (105.0, 89.1), turned to 0 degrees
- moved U4 8.94 mm to (113.2, 81.7)
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Connections:
- C2 pad 1: +VBUS -> +VBUSF
Routing:
- net /NRST: track 0.00 -> 30.7 mm
- net /UART2_TX: track 20.9 -> 2.96 mm
- net Net-(U1-PA5): track 0.00 -> 16.5 mm
- net /UART2_RX: track 15.9 -> 2.92 mm
- net /SWD_IO: track 0.00 -> 9.64 mm
- net /SWD_CLK: track 0.00 -> 8.32 mm
- net Net-(U1-PA6): track 0.00 -> 7.36 mm
- net /VREF+: track 0.00 -> 4.97 mm
- net +3V3: track 0.00 -> 4.88 mm
- net Net-(U1-PA2): track 0.00 -> 4.25 mm
- net /VREF-: track 0.00 -> 4.09 mm
- net GND: track 0.00 -> 3.65 mm, vias 4 -> 5
- net Net-(U1-VCORE): track 0.00 -> 1.60 mm
