File: mspm0-dev-hw/mspm0-dev.kicad_sch (KiCad schematic)
At the start: 33 parts, among them J1 USB_C_Receptacle_USB2.0_14P, J2 Conn_02x05_Odd_Even, J3 TC2030, U1 MSPM0G3507SPTR, U4 SPX3819M5-L-3-3, U5 CH340E, Y1 8MHz

Commit message: bump hardware changes
Parts:
- added FID1, FID2, FID3: Fiducial, Fiducial:Fiducial_0.5mm_Mask1mm, symbol Mechanical:Fiducial
- added H1, H2, H3, H4: MountingHole_Pad, MountingHole:MountingHole_2.5mm_Pad_TopOnly, symbol Mechanical:MountingHole_Pad
- C1, C10, C11, C12, C13, C15, C16, C2, C3, C5, C8, C9: footprint (none) -> Capacitor_SMD:C_0603_1608Metric
- C14, C4, C6: footprint (none) -> Capacitor_SMD:C_0805_2012Metric
- D2: footprint (none) -> LED_SMD:LED_0603_1608Metric
- J1: footprint (none) -> Connector_USB:USB_C_Receptacle_GCT_USB4110
- J2: footprint (none) -> Connector_PinHeader_2.54mm:PinHeader_2x05_P2.54mm_Horizontal
- R1, R2, R3, R4, R5, R6, R8, R9: footprint (none) -> Resistor_SMD:R_0603_1608Metric
- R7: footprint Capacitor_SMD:C_0603_1608Metric_Pad1.08x0.95mm_HandSolder -> Resistor_SMD:R_0603_1608Metric
Connections:
- net GND: now also H1.1, H2.1, H3.1, H4.1
- net I2C1_SCL: now also R8.1
- net I2C1_SDA: now also R9.1
- net A1_0 renamed GPIO_A1_0
- net A1_1 renamed GPIO_A1_1
- net I2C0_SCL: no longer names the net of U1.19 (PA11)
- net I2C0_SCL: no longer R9.1
- net I2C0_SDA: no longer names the net of U1.18 (PA10)
- net I2C0_SDA: no longer R8.1
- net PA_12: no longer names the net of U1.27 (PA12)
- net PA_12: no longer J2.7 (Pin_7)
- net PA_13: no longer names the net of U1.28 (PA13)
- net PA_13: no longer J2.8 (Pin_8)
- new net GPIO_PA26: J2.7 (Pin_7)
- new net GPIO_PA27: J2.8 (Pin_8)
- no-connect marks 22 -> 26

Commit message: begin routing
Parts:
- removed C2: 470n, Capacitor_SMD:C_0603_1608Metric, symbol Device:C
- renumbered C3 to C2
Other:
- moved on the sheet: C2, R3
